File: Hardware/Auto.kicad_sch (KiCad schematic)
At the start: 43 parts, among them J10 M2, J11 M3, J12 M4, J13 DISTANCIA, J9 M1, U5 74HC595, U6 TB6612FNG, U8 TB6612FNG

Commit message: Actualizo a versión 1.4
Parts:
- J10, J11, J12, J9: footprint footprints:CONN2_2060-1452&slash_998-404_WAG -> footprints:691214310002; symbol 2024-09-06_13-56-18:2060-452_998-404 -> Connector_Generic:Conn_01x02; Manufacturer WAGO Corporation -> Würth Elektronik; Package 0.157" (4.00mm) -> 0.150" (3.81mm); PartNumber 2060-1452/998-404 -> 691214310002; PurchaseLink https://www.digikey.com/en/products/detail/wago-corporation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 -> https://www.digikey.com/en/products/detail/w%C3%BCrth-elekt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
Connections:
- net at C16.2, J11.1 (Pin_1), TP24.1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: no longer J11.2 (1_2)
- net at C16.1, TP25.1, U6.5 (AO2)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: now also J11.2 (Pin_2); no longer J11.3 (2_1), J11.4 (2_2)
- net at C24.2, J10.1 (Pin_1), TP20.1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: no longer J10.2 (1_2)
- net at C25.2, TP22.1, U8.11 (BO1)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: now also J9.2 (Pin_2); no longer J9.3 (2_1), J9.4 (2_2)
- net at C24.1, TP21.1, U8.5 (AO2)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: now also J10.2 (Pin_2); no longer J10.3 (2_1), J10.4 (2_2)
- net at C25.1, J9.1 (Pin_1), TP23.1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: no longer J9.2 (1_2)
- net at C17.1, J12.1 (Pin_1), TP27.1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: no longer J12.2 (1_2)
- net at C17.2, TP26.1, U6.11 (BO1)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: now also J12.2 (Pin_2); no longer J12.3 (2_1), J12.4 (2_2)

Commit message: Elimino testpoints de BOM
Parts:
- TP20, TP21, TP22, TP23, TP24, TP25, TP26, TP27, TP32, TP33, TP34, TP35, TP36: now left out of the parts list
Changed lines of the file:
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@@
 		(unit 1)
 		(exclude_from_sim no)
-		(in_bom yes)
+		(in_bom no)
 		(on_board yes)
 		(dnp no)
@@
 		(unit 1)
 		(exclude_from_sim no)
-		(in_bom yes)
+		(in_bom no)
 		(on_board yes)
 		(dnp no)
@@
 		(unit 1)
 		(exclude_from_sim no)
-		(in_bom yes)
+		(in_bom no)
 		(on_board yes)
 		(dnp no)
@@
 		(unit 1)
 		(exclude_from_sim no)
-		(in_bom yes)
+		(in_bom no)
 		(on_board yes)
 		(dnp no)
@@
 		(unit 1)
 		(exclude_from_sim no)
-		(in_bom yes)
+		(in_bom no)
 		(on_board yes)
 		(dnp no)
@@
 		(unit 1)
 		(exclude_from_sim no)
-		(in_bom yes)
+		(in_bom no)
 		(on_board yes)
 		(dnp no)
@@
 		(unit 1)
 		(exclude_from_sim no)
-		(in_bom yes)
+		(in_bom no)
 		(on_board yes)
 		(dnp no)
@@
 			)
 		)
+		(property "PartNumber" ""
+			(at 166.37 55.88 0)
+			(effects
+				(font
+					(size 1.27 1.27)
+				)
+				(hide yes)
+			)
+		)
+		(property "PurchaseLink" ""
+			(at 166.37 55.88 0)
+			(effects
+				(font
+					(size 1.27 1.27)
+				)
+				(hide yes)
+			)
+		)
 		(pin "1"
 		)
@@
 		(unit 1)
 		(exclude_from_sim no)
-		(in_bom yes)
+		(in_bom no)
 		(on_board yes)
 		(dnp no)
@@
 		(unit 1)
 		(exclude_from_sim no)
-		(in_bom yes)
+		(in_bom no)
 		(on_board yes)
 		(dnp no)
@@
 		(unit 1)
 		(exclude_from_sim no)
-		(in_bom yes)
+		(in_bom no)
 		(on_board yes)
 		(dnp no)
@@
 		(unit 1)
 		(exclude_from_sim no)
-		(in_bom yes)
+		(in_bom no)
 		(on_board yes)
 		(dnp no)
@@
 		(unit 1)
 		(exclude_from_sim no)
-		(in_bom yes)
+		(in_bom no)
 		(on_board yes)
 		(dnp no)
@@
 		(unit 1)
 		(exclude_from_sim no)
-		(in_bom yes)
+		(in_bom no)
 		(on_board yes)
 		(dnp no)
