File: Hardware/Power.kicad_sch (KiCad schematic)
At the start: 25 parts, among them J1 BAT, U1 TPS563252DRLR

Commit message: Actualizo a versión 1.4
Parts:
- J1: footprint footprints:CONN2_2060-1452&slash_998-404_WAG -> footprints:691214310002; symbol 2024-09-06_13-56-18:2060-452_998-404 -> Connector_Generic:Conn_01x02; Manufacturer WAGO Corporation -> Würth Elektronik; Package 0.157" (4.00mm) -> 0.150" (3.81mm); PartNumber 2060-1452/998-404 -> 691214310002; PurchaseLink https://www.digikey.com/en/products/detail/wago-corporation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 -> https://www.digikey.com/en/products/detail/w%C3%BCrth-elekt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
Connections:
- net GND: no longer J1.2 (1_2)
- net VBAT: now also J1.2 (Pin_2); no longer J1.3 (2_1), J1.4 (2_2)
Changed lines of the file:
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@@
 	(title_block
 		(title "Archi Bot")
-		(date "2025-05-28")
-		(rev "1.3")
+		(date "2025-06-11")
+		(rev "1.4")
 		(company "Newsan")
 	)
@@
 	)
 	(junction
-		(at 74.93 135.89)
-		(diameter 0)
-		(color 0 0 0 0)
-	)
-	(junction
 		(at 74.93 140.97)
 		(diameter 0)
@@
 	)
 	(junction
-		(at 74.93 143.51)
-		(diameter 0)
-		(color 0 0 0 0)
-	)
-	(junction
 		(at 106.68 147.32)
 		(diameter 0)
@@
 	(wire
 		(pts
-			(xy 74.93 143.51) (xy 74.93 144.78)
+			(xy 74.93 140.97) (xy 74.93 142.24)
 		)
 		(stroke
@@
 	(wire
 		(pts
-			(xy 74.93 138.43) (xy 74.93 135.89)
+			(xy 74.93 137.16) (xy 74.93 138.43)
 		)
 		(stroke
@@
 	(wire
 		(pts
-			(xy 73.66 143.51) (xy 74.93 143.51)
-		)
-		(stroke
-			(width 0)
-			(type default)
-		)
-	)
-	(wire
-		(pts
 			(xy 106.68 138.43) (xy 106.68 137.16)
 		)
@@
 	(wire
 		(pts
-			(xy 74.93 140.97) (xy 74.93 143.51)
-		)
-		(stroke
-			(width 0)
-			(type default)
-		)
-	)
-	(wire
-		(pts
-			(xy 74.93 135.89) (xy 74.93 134.62)
-		)
-		(stroke
-			(width 0)
-			(type default)
-		)
-	)
-	(wire
-		(pts
 			(xy 157.48 118.11) (xy 158.75 118.11)
 		)
@@
 		)
 	)
-	(wire
-		(pts
-			(xy 73.66 135.89) (xy 74.93 135.89)
-		)
-		(stroke
-			(width 0)
-			(type default)
-		)
-	)
 	(polyline
 		(pts
@@
 			"AAAAAAAAAAAAAAAAAAAAAAChbR0AAQAAAAAAAAAAAAAAAAAAAAAAAAAAAAAAAAAAAAAAAAAAAAAA"
 			"kPIJAAEAAAAAAAAAAAAAAAAAAAAAAAAAAAAAAAAAAAAAAAAAAAAAAN2BagABrLoDAAAAAAAAAAAA"
-			"AAAAAAAAAAAAAAAAAAAAAAAAAAAAAA=="
+			"AAAAAAAAAAAAAAAAAAAAAAAAAAAAAIBUZXJtaW5hbAAAAAAAAAAAAAAAAAAAAAB1KqPnAFAEgAAA"
+			"AAAAAAAAfHzGnQAAAABAwHJuYwEAAHsqoecAUQSABgAAABAAAABw0gAAAAAAAAAAAAAAAAAAeSqv"
+			"5wBSBIBTdGFuZGFyZAAAAAAAAAAAAAAAAAAAAAB/Kq3nAFMEgE5vcm1hYWxpAAAAAAAAAAAAAAAA"
+			"AAAAAH0qq+cAVASABgAAABAAAACAtwAAAAAAAAAAAAAAAAAAAyqp5wBVBIBZdSBHb3RoaWMgVUkA"
+			"AAAAAAAAAAAAAAABKtfnAFYEgG9iecSNZWpuw6kAAAAAAAAAAAAAAAAAAAcq1ecAVwSAAAAAAAAA"
+			"AABCJmimAAAAAKDAcm5jAQAABSrT5wBYBIAGAAAAEAAAAACVAAAAAAAAAAAAAAAAAAALKtHnAFkE"
+			"gFN0YW5kYWFyZAAAAAAAAAAAAAAAAAAAAAkq3+cAWgSATm9ybWFsbnkAAAAAAAAAAAAAAAAAAAAA"
+			"Dyrd5wBbBIBZdSBHb3RoaWMAAAAAAAAAAAAAAAAAAAANKtvnAFwEgAYAAAAQAAAAMMIAAAAAAAAA"
+			"AAAAAAAAABMq2ecAXQSAzprOsc69zr/Ovc65zrrOrAAAAAAAAAAAESrH5wBeBIDQntCx0YvRh9C9"
+			"0YvQuQAAAAAAAAAAAAAXKsXnAF8EgE5vcm3DoWxuZQAAAAAAAAAAAAAAAAAAABUqw+cAYASAdGjG"
+			"sMahzIBuZwAAAAAAAAAAAAAAAAAAGyrB5wBhBIAAAAAAAAAAABLq2tMAAAAAwL1ybmMBAAAZKs/n"
+			"AGIEgAYAAAAQAAAAkNQAAAAAAAAAAAAAAAAAAB8qzecAYwSAzojOvc+Ezr/Ovc6xAAAAAAAAAAAA"
+			"AAAAHSrL5wBkBIBMaWhhdm9pdHUAAAAAAAAAAAAAAAAAAAAjKsnnAGUEgEbDqWxrw7Z2w6lyAAAA"
+			"AAAAAAAAAAAAACEq9+cAZgSAR3Jhc3NldHRvAAAAAAAAAAAAAAAAAAAAJyr15wBnBIBQb2dydWJp"
+			"b255AAAAAAAAAAAAAAAAAAAlKvPnAGgEgNCf0L7Qu9GD0LbQuNGA0L3Ri9C5AAAAACsq8ecAaQSA"
+			"AAAAAAAAAAAUSUW+AAAAAMC+cm5jAQAAKSr/5wBqBIAGAAAAEAAAAGDQAAAAAAAAAAAAAAAAAAAv"
+			"Kv3nAGsEgAAAAAAAAAAAYseLdgAAAAAAvXJuYwEAAC0q++cAbASAQm9sZCBJdGFsaWMAAAAAAAAA"
+			"AAAAAAAAMyr55wBtBIAGAAAAEAAAAHC1AAAAAAAAAAAAAAAAAAAxKufnAG4EgE5lZ3JldGEgY3Vy"
+			"c2l2YQAAAAAAAAAAADcq5ecAbwSAVA=="
 		)
 	)
@@
 			"8qcGAPOnBgD0pwYA9acGAPanBgD3pwYA+KcGAPmnBgD6pwYA+6cGAPynBgD9pwYA/qcGAP+nBgAA"
 			"qAYAAagGAAKoBgADqAYABKgGAAWoBgAGqAYAB6gGAAioBgAJqAYACqgGAAuoBgAMqAYADagGAA6o"
-			"BgAPqAYAEKgGABGoBgASqAYAE6gGAA=="
+			"BgAPqAYAEKgGABGoBgASqAYAE6gGAAAAAAAAAAAAAAAAAAAAAAAAAAAAAAAAAAAAAAAAAAAAAAAA"
+			"AAAAAAAAAAAAAAAAAAAAAAAAAAAAAAAAAAAAAAAAAAAAAAAAAAAAAAAAAAAAAAAAAAAAAAAAAAAA"
+			"AAAAAAAAAAAAAAAAAAAAAAAAAAAAAAAAAAAAAAAAAAAAAAAAAAAAAAAAAAAAAAAAAAAAAAAAAAAA"
+			"AAAAAAAAAAAAAAAAAAAAAAAAAAAAAAAAAAAAAAAAAAAAAAAAAAAAAAAAAAAAAAAAAAAAAAAAAAAA"
+			"AAAAAAAAAAAAAAAAAAAAAAAAAAAAAAAAAAAAAAAAAAAAAAAAAAAAAAAAAAAAAAAAAAAAAAAAAAAA"
+			"AAAAAAAAAAAAAAAAAAAAAAAAAAAAAAAAAAAAAAAAAAAAAAAAAAAAAAAAAAAAAAAAAAAAAAAAAAAA"
+			"AAAAAAAAAAAAAAAAAAAAAAAAAAAAAAAAAAAAAAAAAAAAAAAAAAAAAAAAAAAAAAAAAAAAAAAAAAAA"
+			"AAAAAAAAAAAAAAAAAAAAAAAAAAAAAAAAAAAAAAAAAAAAAAAAAAAAAAAAAAAAAAAAAAAAAAAAAAAA"
+			"AAAAAAAAAAAAAAAAAAAAAAAAAAAAAAAAAAAAAAAAAAAAAAAAAAAAAAAAAAAAAAAAAAAAAAAAAAAA"
+			"AAAAAAAAAAAAAAAAAAAAAAAAAAAAAAAAAAAAAAAAAAAAAAAAAAAAAAAAAAAAAAAAAAAAAAAAAAAA"
+			"AAAAAAAAAAAAAAAAAAAAAAAAAAAAAAAAAAAAAAAAAAAAAAAAAAAAAAAAAAAAAAAAAAAAAAAAAAAA"
+			"AAAAAAAAAAAAAAAAAAAAAAAAAAAAAAAAAAAAAAAAAAAAAAAAAAAAAAAAAAAAAAAAAAAAAAAAAAAA"
+			"AAAAAAAAAAAAAAAAAAAAAAAAAAAAAAAAAAAAAAAAAAAAAAAAAAAAAAAAAAAAAAAAAAAAAAAAAAAA"
+			"AAAAAAAAAAAAAAAAAAAAAAAAAAAAAAAAAAAAAAAAAAAAAAAAAAAAAAAAAAAAAAAAAAAAAAAAAAAA"
+			"AAAAAAAAAAAAAAAAAAAAAAAAAAAAAAAAAAAAAAAAAAAAAAAAAAAAAAAAAAAAAAAAAAAAAAAAAAAA"
+			"AAAAAAAAAAAAAAAAAAAAAAAAAAAAAAAAAAAAAAAAAAAAAAAAAAAAAAAAAAAAAAAAAAAAAAAAAAAA"
+			"AAAAAAAAAAAAAAAAAAAAAAAAAAAAAAAAAAAAAAAAAAAAAAAAAAAAAAAAAAAAAAAAAAAAAAAAAAAA"
+			"AAAAAAAAAAAAAAAAAAAAAAAAAAAAAAAAAAAAAAAAAAAAAAAAAAAAAAAAAAAAAAAAAAAAAAAAAAAA"
+			"AAAAAAAAAAAAAAAAAAAAAAAAAAAAAA=="
 		)
 	)
@@
 	)
 	(symbol
-		(lib_id "2024-09-06_13-56-18:2060-452_998-404")
-		(at 73.66 143.51 180)
+		(lib_id "Connector_Generic:Conn_01x02")
+		(at 68.58 140.97 180)
 		(unit 1)
 		(exclude_from_sim no)
@@
 		(dnp no)
 		(property "Reference" "J1"
-			(at 67.31 129.54 0)
+			(at 68.58 133.604 0)
 			(effects
 				(font
@@
 		)
 		(property "Value" "BAT"
-			(at 67.31 132.08 0)
+			(at 68.58 136.144 0)
 			(effects
 				(font
@@
 			)
 		)
-		(property "Footprint" "footprints:CONN2_2060-1452&slash_998-404_WAG"
-			(at 73.66 143.51 0)
+		(property "Footprint" "footprints:691214310002"
+			(at 68.58 140.97 0)
 			(effects
 				(font
 					(size 1.27 1.27)
-					(italic yes)
 				)
 				(hide yes)
 			)
 		)
-		(property "Datasheet" "https://www.wago.com/global/pcb-terminal-blocks-and-pluggable-connectors/thr-terminal-block-with-push-buttons-in-tape-and-reel-packing/p/2060-1452_998-404"
-			(at 73.66 143.51 0)
+		(property "Datasheet" "https://www.we-online.com/catalog/datasheet/691214310002.pdf"
+			(at 68.58 140.97 0)
 			(effects
 				(font
 					(size 1.27 1.27)
-					(italic yes)
 				)
 				(hide yes)
 			)
 		)
-		(property "Description" "THR PCB TERMINAL BLOCK PUSH-BUT 4MM"
-			(at 76.2 143.51 0)
+		(property "Description" "TERM BLK 2POS SIDE ENT 3.81MM HOR"
+			(at 68.58 140.97 0)
 			(effects
 				(font
@@
 			)
 		)
-		(property "PartNumber" "2060-1452/998-404"
-			(at 73.66 143.51 0)
+		(property "PartNumber" "691214310002"
+			(at 68.58 140.97 0)
 			(effects
 				(font
@@
 			)
 		)
-		(property "PurchaseLink" "https://www.digikey.com/en/products/detail/wago-corporation/2060-452-998-404/15540283"
-			(at 73.66 143.51 0)
+		(property "PurchaseLink" "https://www.digikey.com/en/products/detail/w%C3%BCrth-elektronik/691214310002/11477478"
+			(at 68.58 140.97 0)
 			(effects
 				(font
@@
 			)
 		)
-		(property "Manufacturer" "WAGO Corporation"
-			(at 73.66 143.51 0)
+		(property "Manufacturer" "Würth Elektronik"
+			(at 68.58 140.97 0)
 			(effects
 				(font
@@
 			)
 		)
-		(property "Package" "0.157\" (4.00mm)"
-			(at 73.66 143.51 0)
+		(property "Package" "0.150\" (3.81mm)"
+			(at 68.58 140.97 0)
 			(effects
 				(font
@@
 		(pin "2"
 		)
-		(pin "4"
-		)
-		(pin "3"
-		)
 		(instances
 			(project "ArchiBot"
@@
 	(symbol
 		(lib_id "power:GND")
-		(at 74.93 144.78 0)
+		(at 74.93 142.24 0)
 		(unit 1)
 		(exclude_from_sim no)
@@
 		(dnp no)
 		(property "Reference" "#PWR02"
-			(at 74.93 151.13 0)
+			(at 74.93 148.59 0)
 			(effects
 				(font
@@
 		)
 		(property "Value" "GND"
-			(at 74.93 148.59 0)
+			(at 74.93 146.05 0)
 			(effects
 				(font
@@
 		)
 		(property "Footprint" ""
-			(at 74.93 144.78 0)
+			(at 74.93 142.24 0)
 			(effects
 				(font
@@
 		)
 		(property "Datasheet" ""
-			(at 74.93 144.78 0)
+			(at 74.93 142.24 0)
 			(effects
 				(font
@@
 		)
 		(property "Description" ""
-			(at 74.93 144.78 0)
+			(at 74.93 142.24 0)
 			(effects
 				(font
@@
 	(symbol
 		(lib_id "power:VBUS")
-		(at 74.93 134.62 0)
+		(at 74.93 137.16 0)
 		(unit 1)
 		(exclude_from_sim no)
@@
 		(dnp no)
 		(property "Reference" "#PWR01"
-			(at 74.93 138.43 0)
+			(at 74.93 140.97 0)
 			(effects
 				(font
@@
 		)
 		(property "Value" "VBAT"
-			(at 74.93 131.318 0)
+			(at 74.93 133.858 0)
 			(effects
 				(font
@@
 		)
 		(property "Footprint" ""
-			(at 74.93 134.62 0)
+			(at 74.93 137.16 0)
 			(effects
 				(font
@@
 		)
 		(property "Datasheet" ""
-			(at 74.93 134.62 0)
+			(at 74.93 137.16 0)
 			(effects
 				(font
@@
 		)
 		(property "Description" "Power symbol creates a global label with name \"VBUS\""
-			(at 74.93 134.62 0)
+			(at 74.93 137.16 0)
 			(effects
 				(font

Commit message: Elimino testpoints de BOM
Parts:
- TP1, TP2, TP3, TP37, TP38: now left out of the parts list
Changed lines of the file:
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@@
 		(unit 1)
 		(exclude_from_sim no)
-		(in_bom yes)
+		(in_bom no)
 		(on_board yes)
 		(dnp no)
@@
 			)
 		)
+		(property "PartNumber" ""
+			(at 166.37 135.89 0)
+			(effects
+				(font
+					(size 1.27 1.27)
+				)
+				(hide yes)
+			)
+		)
+		(property "PurchaseLink" ""
+			(at 166.37 135.89 0)
+			(effects
+				(font
+					(size 1.27 1.27)
+				)
+				(hide yes)
+			)
+		)
 		(pin "1"
 		)
@@
 		(unit 1)
 		(exclude_from_sim no)
-		(in_bom yes)
+		(in_bom no)
 		(on_board yes)
 		(dnp no)
@@
 		(unit 1)
 		(exclude_from_sim no)
-		(in_bom yes)
+		(in_bom no)
 		(on_board yes)
 		(dnp no)
@@
 			)
 		)
+		(property "PartNumber" ""
+			(at 78.74 137.16 0)
+			(effects
+				(font
+					(size 1.27 1.27)
+				)
+				(hide yes)
+			)
+		)
+		(property "PurchaseLink" ""
+			(at 78.74 137.16 0)
+			(effects
+				(font
+					(size 1.27 1.27)
+				)
+				(hide yes)
+			)
+		)
 		(pin "1"
 		)
@@
 		(unit 1)
 		(exclude_from_sim no)
-		(in_bom yes)
+		(in_bom no)
 		(on_board yes)
 		(dnp no)
@@
 			)
 		)
+		(property "PartNumber" ""
+			(at 81.28 137.16 0)
+			(effects
+				(font
+					(size 1.27 1.27)
+				)
+				(hide yes)
+			)
+		)
+		(property "PurchaseLink" ""
+			(at 81.28 137.16 0)
+			(effects
+				(font
+					(size 1.27 1.27)
+				)
+				(hide yes)
+			)
+		)
 		(pin "1"
 		)
@@
 		(unit 1)
 		(exclude_from_sim no)
-		(in_bom yes)
-		(on_board yes)
-		(dnp no)
+		(in_bom no)
+		(on_board yes)
+		(dnp no)
